File: PCB/Postmaster/ethernet.kicad_sch (KiCad schematic)
At the start: 33 parts, among them P1 J00-0065NL, U1 LAN8710A

Commit message: Update schematics
Changed lines of the file:
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@@
+	)
+	(junction
+		(at 193.04 29.21)
+		(diameter 0)
+		(color 0 0 0 0)
 	)
 	(junction
@@
 		(shape output)
 		(at 255.27 81.28 0)
-		(fields_autoplaced yes)
 		(effects
 			(font
@@
 		(shape input)
 		(at 210.82 66.04 0)
-		(fields_autoplaced yes)
 		(effects
 			(font
@@
 		(shape input)
 		(at 255.27 101.6 0)
-		(fields_autoplaced yes)
 		(effects
 			(font
@@
 		(shape output)
 		(at 255.27 83.82 0)
-		(fields_autoplaced yes)
 		(effects
 			(font
@@
 		(shape bidirectional)
 		(at 276.86 109.22 0)
-		(fields_autoplaced yes)
 		(effects
 			(font
@@
 		(shape input)
 		(at 210.82 73.66 0)
-		(fields_autoplaced yes)
 		(effects
 			(font
@@
 		(shape input)
 		(at 276.86 111.76 0)
-		(fields_autoplaced yes)
 		(effects
 			(font
@@
 		(shape input)
 		(at 210.82 63.5 0)
-		(fields_autoplaced yes)
 		(effects
 			(font
@@
 		(shape input)
 		(at 210.82 121.92 0)
-		(fields_autoplaced yes)
 		(effects
 			(font
@@
 			)
 			(justify left)
+		)
+	)
+	(symbol
+		(lib_id "power:PWR_FLAG")
+		(at 187.96 45.72 0)
+		(unit 1)
+		(exclude_from_sim no)
+		(in_bom yes)
+		(on_board yes)
+		(dnp no)
+		(fields_autoplaced yes)
+		(property "Reference" "#FLG04"
+			(at 187.96 43.815 0)
+			(effects
+				(font
+					(size 1.27 1.27)
+				)
+				(hide yes)
+			)
+		)
+		(property "Value" "PWR_FLAG"
+			(at 187.96 40.64 0)
+			(effects
+				(font
+					(size 1.27 1.27)
+				)
+			)
+		)
+		(property "Footprint" ""
+			(at 187.96 45.72 0)
+			(effects
+				(font
+					(size 1.27 1.27)
+				)
+				(hide yes)
+			)
+		)
+		(property "Datasheet" "~"
+			(at 187.96 45.72 0)
+			(effects
+				(font
+					(size 1.27 1.27)
+				)
+				(hide yes)
+			)
+		)
+		(property "Description" "Special symbol for telling ERC where power comes from"
+			(at 187.96 45.72 0)
+			(effects
+				(font
+					(size 1.27 1.27)
+				)
+				(hide yes)
+			)
+		)
+		(pin "1"
+		)
+		(instances
+			(project "Postmaster"
+				(path "/b2fb7ca8-b44b-45c2-b25e-cd50f2bbc5c4/c4600c43-5b92-49d3-8115-df606fc80505"
+					(reference "#FLG04")
+					(unit 1)
+				)
+			)
 		)
 	)
@@
 					(unit 1)
 				)
+			)
+		)
+	)
+	(symbol
+		(lib_id "power:PWR_FLAG")
+		(at 193.04 29.21 0)
+		(unit 1)
+		(exclude_from_sim no)
+		(in_bom yes)
+		(on_board yes)
+		(dnp no)
+		(fields_autoplaced yes)
+		(property "Reference" "#FLG03"
+			(at 193.04 27.305 0)
+			(effects
+				(font
+					(size 1.27 1.27)
+				)
+				(hide yes)
+			)
+		)
+		(property "Value" "PWR_FLAG"
+			(at 193.04 24.13 0)
+			(effects
+				(font
+					(size 1.27 1.27)
+				)
+			)
+		)
+		(property "Footprint" ""
+			(at 193.04 29.21 0)
+			(effects
+				(font
+					(size 1.27 1.27)
+				)
+				(hide yes)
+			)
+		)
+		(property "Datasheet" "~"
+			(at 193.04 29.21 0)
+			(effects
+				(font
+					(size 1.27 1.27)
+				)
+				(hide yes)
+			)
+		)
+		(property "Description" "Special symbol for telling ERC where power comes from"
+			(at 193.04 29.21 0)
+			(effects
+				(font
+					(size 1.27 1.27)
+				)
+				(hide yes)
+			)
+		)
+		(pin "1"
+		)
+		(instances
+			(project "Postmaster"
+				(path "/b2fb7ca8-b44b-45c2-b25e-cd50f2bbc5c4/c4600c43-5b92-49d3-8115-df606fc80505"
+					(reference "#FLG03")
+					(unit 1)
+				)

Commit message: Update schematics
Other:
- moved on the sheet: R2
Changed lines of the file:
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@@
 	(wire
 		(pts
-			(xy 269.24 109.22) (xy 276.86 109.22)
+			(xy 269.24 109.22) (xy 274.32 109.22)
 		)
 		(stroke
@@
 	(wire
 		(pts
+			(xy 212.09 121.92) (xy 210.82 121.92)
+		)
+		(stroke
+			(width 0)
+			(type default)
+		)
+	)
+	(wire
+		(pts
 			(xy 92.71 73.66) (xy 92.71 45.72)
 		)
@@
 	(wire
 		(pts
+			(xy 29.21 137.16) (xy 29.21 138.43)
+		)
+		(stroke
+			(width 0)
+			(type default)
+		)
+	)
+	(wire
+		(pts
 			(xy 236.22 45.72) (xy 245.11 45.72)
 		)
@@
 	(wire
 		(pts
+			(xy 212.09 73.66) (xy 210.82 73.66)
+		)
+		(stroke
+			(width 0)
+			(type default)
+		)
+	)
+	(wire
+		(pts
 			(xy 124.46 45.72) (xy 134.62 45.72)
 		)
@@
 	(wire
 		(pts
-			(xy 210.82 111.76) (xy 276.86 111.76)
+			(xy 212.09 63.5) (xy 210.82 63.5)
+		)
+		(stroke
+			(width 0)
+			(type default)
+		)
+	)
+	(wire
+		(pts
+			(xy 210.82 111.76) (xy 274.32 111.76)
 		)
 		(stroke
@@
 	(wire
 		(pts
+			(xy 212.09 66.04) (xy 210.82 66.04)
+		)
+		(stroke
+			(width 0)
+			(type default)
+		)
+	)
+	(wire
+		(pts
 			(xy 201.93 45.72) (xy 205.74 45.72)
 		)
@@
 	(wire
 		(pts
-			(xy 29.21 124.46) (xy 29.21 132.08)
+			(xy 29.21 124.46) (xy 29.21 129.54)
 		)
 		(stroke
@@
 		(pts
 			(xy 254 101.6) (xy 254 53.34)
-		)
-		(stroke
-			(width 0)
-			(type default)
-		)
-	)
-	(wire
-		(pts
-			(xy 29.21 132.08) (xy 81.28 132.08)
 		)
 		(stroke
@@
 		(shape output)
 		(at 255.27 81.28 0)
+		(fields_autoplaced yes)
 		(effects
 			(font
@@
 	(hierarchical_label "txd1"
 		(shape input)
-		(at 210.82 66.04 0)
+		(at 212.09 66.04 0)
+		(fields_autoplaced yes)
 		(effects
 			(font
@@
 		(shape input)
 		(at 255.27 101.6 0)
+		(fields_autoplaced yes)
 		(effects
 			(font
@@
 		(shape output)
 		(at 255.27 83.82 0)
+		(fields_autoplaced yes)
 		(effects
 			(font
@@
 	(hierarchical_label "mdio"
 		(shape bidirectional)
-		(at 276.86 109.22 0)
+		(at 274.32 109.22 0)
+		(fields_autoplaced yes)
 		(effects
 			(font
@@
 	(hierarchical_label "txen"
 		(shape input)
-		(at 210.82 73.66 0)
+		(at 212.09 73.66 0)
+		(fields_autoplaced yes)
 		(effects
 			(font
@@
 	(hierarchical_label "mdc"
 		(shape input)
-		(at 276.86 111.76 0)
+		(at 274.32 111.76 0)
+		(fields_autoplaced yes)
 		(effects
 			(font
@@
 	(hierarchical_label "txd0"
 		(shape input)
-		(at 210.82 63.5 0)
+		(at 212.09 63.5 0)
+		(fields_autoplaced yes)
 		(effects
 			(font
@@
 	(hierarchical_label "clkin"
 		(shape input)
-		(at 210.82 121.92 0)
+		(at 212.09 121.92 0)
+		(fields_autoplaced yes)
 		(effects
 			(font
@@
 	(symbol
 		(lib_id "Device:R")
-		(at 81.28 135.89 0)
+		(at 29.21 133.35 0)
 		(unit 1)
 		(exclude_from_sim no)
@@
 		(fields_autoplaced yes)
 		(property "Reference" "R2"
-			(at 83.82 134.6199 0)
+			(at 31.75 132.0799 0)
 			(effects
 				(font
@@
 		)
 		(property "Value" "330"
-			(at 83.82 137.1599 0)
+			(at 31.75 134.6199 0)
 			(effects
 				(font
@@
 		)
 		(property "Footprint" "Resistor_SMD:R_0603_1608Metric"
-			(at 79.502 135.89 90)
+			(at 27.432 133.35 90)
 			(effects
 				(font
@@
 		)
 		(property "Datasheet" "~"
-			(at 81.28 135.89 0)
+			(at 29.21 133.35 0)
 			(effects
 				(font
@@
 		)
 		(property "Description" "Resistor"
-			(at 81.28 135.89 0)
+			(at 29.21 133.35 0)
 			(effects
 				(font
@@
 		)
 		(property "JLCPCBPart" "C23138"
-			(at 81.28 135.89 0)
+			(at 29.21 133.35 0)
 			(effects
 				(font
@@
 	(symbol
 		(lib_id "power:GND")
-		(at 81.28 139.7 0)
+		(at 29.21 138.43 0)
 		(unit 1)
 		(exclude_from_sim no)
@@
 		(fields_autoplaced yes)
 		(property "Reference" "#PWR01"
-			(at 81.28 146.05 0)
+			(at 29.21 144.78 0)
 			(effects
 				(font
@@
 		)
 		(property "Value" "GND"
-			(at 81.28 144.78 0)
+			(at 29.21 143.51 0)
 			(effects
 				(font
@@
 		)
 		(property "Footprint" ""
-			(at 81.28 139.7 0)
+			(at 29.21 138.43 0)
 			(effects
 				(font
@@
 		)
 		(property "Datasheet" ""
-			(at 81.28 139.7 0)
+			(at 29.21 138.43 0)
 			(effects
 				(font
@@
 		)
 		(property "Description" "Power symbol creates a global label with name \"GND\" , ground"
-			(at 81.28 139.7 0)
-			(effects
-				(font
+			(at 29.21 138.43 0)
+			(effects
+				(font

Commit message: Update schematics
Parts:
- P1: footprint J00-0065NL:PULSE_J00-0065NL -> PostmasterParts:PULSE_J00-0065NL
Changed lines of the file:
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@@
 		(shape output)
 		(at 255.27 81.28 0)
-		(fields_autoplaced yes)
 		(effects
 			(font
@@
 		(shape input)
 		(at 212.09 66.04 0)
-		(fields_autoplaced yes)
 		(effects
 			(font
@@
 		(shape input)
 		(at 255.27 101.6 0)
-		(fields_autoplaced yes)
 		(effects
 			(font
@@
 		(shape output)
 		(at 255.27 83.82 0)
-		(fields_autoplaced yes)
 		(effects
 			(font
@@
 		(shape bidirectional)
 		(at 274.32 109.22 0)
-		(fields_autoplaced yes)
 		(effects
 			(font
@@
 		(shape input)
 		(at 212.09 73.66 0)
-		(fields_autoplaced yes)
 		(effects
 			(font
@@
 		(shape input)
 		(at 274.32 111.76 0)
-		(fields_autoplaced yes)
 		(effects
 			(font
@@
 		(shape input)
 		(at 212.09 63.5 0)
-		(fields_autoplaced yes)
 		(effects
 			(font
@@
 		(shape input)
 		(at 212.09 121.92 0)
-		(fields_autoplaced yes)
 		(effects
 			(font
@@
 			)
 		)
-		(property "Footprint" "J00-0065NL:PULSE_J00-0065NL"
+		(property "Footprint" "PostmasterParts:PULSE_J00-0065NL"
 			(at 49.53 91.44 0)
 			(effects

Commit message: Update schematics, add production files
Parts:
- C2, C3, C4, C5: JCLPCBPart C1634 -> (none); JLCPCBPart (none) -> C1634
- P1: Check_prices https://www.snapeda.com/parts/J00-0065NL/Pulse/view-part/?r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 -> (none); Description_1 1 Port RJ45Through Hole 10/100 Base-TX, AutoMDIX -> (none); MANUFACTURER Pulse -> (none); MF Pulse Electronics Network -> (none); MP J00-0065NL -> (none); Package None -> (none); Price None -> (none); SnapEDA_Link https://www.snapeda.com/parts/J00-0065NL/Pulse/view-part/?r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 -> (none)
Changed lines of the file:
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@@
 		(shape output)
 		(at 255.27 81.28 0)
+		(fields_autoplaced yes)
 		(effects
 			(font
@@
 		(shape input)
 		(at 212.09 66.04 0)
+		(fields_autoplaced yes)
 		(effects
 			(font
@@
 		(shape input)
 		(at 255.27 101.6 0)
+		(fields_autoplaced yes)
 		(effects
 			(font
@@
 		(shape output)
 		(at 255.27 83.82 0)
+		(fields_autoplaced yes)
 		(effects
 			(font
@@
 		(shape bidirectional)
 		(at 274.32 109.22 0)
+		(fields_autoplaced yes)
 		(effects
 			(font
@@
 		(shape input)
 		(at 212.09 73.66 0)
+		(fields_autoplaced yes)
 		(effects
 			(font
@@
 		(shape input)
 		(at 274.32 111.76 0)
+		(fields_autoplaced yes)
 		(effects
 			(font
@@
 		(shape input)
 		(at 212.09 63.5 0)
+		(fields_autoplaced yes)
 		(effects
 			(font
@@
 		(shape input)
 		(at 212.09 121.92 0)
+		(fields_autoplaced yes)
 		(effects
 			(font
@@
 			)
 		)
-		(property "JCLPCBPart" "C1634"
+		(property "JLCPCBPart" "C1634"
 			(at 134.62 107.95 0)
 			(effects
@@
 			)
 		)
-		(property "MF" "Pulse Electronics Network"
-			(at 49.53 91.44 0)
-			(effects
-				(font
-					(size 1.27 1.27)
-				)
-				(justify bottom)
-				(hide yes)
-			)
-		)
-		(property "Description_1" "\n                        \n                            1 Port RJ45Through Hole 10/100 Base-TX, AutoMDIX\n                        \n"
-			(at 49.53 91.44 0)
-			(effects
-				(font
-					(size 1.27 1.27)
-				)
-				(justify bottom)
-				(hide yes)
-			)
-		)
-		(property "Package" "None"
-			(at 49.53 91.44 0)
-			(effects
-				(font
-					(size 1.27 1.27)
-				)
-				(justify bottom)
-				(hide yes)
-			)
-		)
-		(property "Price" "None"
-			(at 49.53 91.44 0)
-			(effects
-				(font
-					(size 1.27 1.27)
-				)
-				(justify bottom)
-				(hide yes)
-			)
-		)
-		(property "Check_prices" "https://www.snapeda.com/parts/J00-0065NL/Pulse/view-part/?ref=eda"
-			(at 49.53 91.44 0)
-			(effects
-				(font
-					(size 1.27 1.27)
-				)
-				(justify bottom)
-				(hide yes)
-			)
-		)
-		(property "SnapEDA_Link" "https://www.snapeda.com/parts/J00-0065NL/Pulse/view-part/?ref=snap"
-			(at 49.53 91.44 0)
-			(effects
-				(font
-					(size 1.27 1.27)
-				)
-				(justify bottom)
-				(hide yes)
-			)
-		)
-		(property "MP" "J00-0065NL"
-			(at 49.53 91.44 0)
-			(effects
-				(font
-					(size 1.27 1.27)
-				)
-				(justify bottom)
-				(hide yes)
-			)
-		)
 		(property "Availability" "In Stock"
 			(at 49.53 91.44 0)
@@
 			)
 		)
-		(property "MANUFACTURER" "Pulse"
-			(at 49.53 91.44 0)
-			(effects
-				(font
-					(size 1.27 1.27)
-				)
-				(justify bottom)
-				(hide yes)
-			)
-		)
 		(property "JLCPCBPart" "C3178480"
 			(at 49.53 91.44 0)
@@
 			)
 		)
-		(property "JCLPCBPart" "C1634"
+		(property "JLCPCBPart" "C1634"
 			(at 114.3 107.95 0)
 			(effects
@@
 			)
 		)
-		(property "JCLPCBPart" "C1634"
+		(property "JLCPCBPart" "C1634"
 			(at 104.14 107.95 0)
 			(effects
@@
 			)
 		)
-		(property "JCLPCBPart" "C1634"
+		(property "JLCPCBPart" "C1634"
 			(at 124.46 107.95 0)
 			(effects
